Commit message: Update LIMO Gazebo bringup, xacros, and URDF/launch configs

File: src/limo_ros2/limo_car/gazebo/ackermann.xacro (robot description, xacro)
@@ -306,33 +306,26 @@
         <!-- *********************************************************************************************** -->
         <gazebo>
-            <plugin name="gazebo_ros_control" filename="libgazebo_ros_control.so" />
-            <plugin name="ackermann_controller" filename="libgazebo_ros_ackermann_drive.so">
+            <plugin name="gz::sim::systems::AckermannSteering"
+                    filename="libgz-sim-ackermann-steering-system.so">
                 <update_rate>100</update_rate>
+                <!-- Wheels -->
                 <front_left_joint>front_left_wheel_joint</front_left_joint>
                 <front_right_joint>front_right_wheel_joint</front_right_joint>
                 <rear_left_joint>rear_left_wheel_joint</rear_left_joint>
                 <rear_right_joint>rear_right_wheel_joint</rear_right_joint>
+                <!-- Steering -->
                 <left_steering_joint>front_left_steer_joint</left_steering_joint>
                 <right_steering_joint>front_right_steer_joint</right_steering_joint>
-                <steering_wheel_joint>/</steering_wheel_joint>
-                <left_steering_pid_gain>10000 100 10</left_steering_pid_gain>
-                <left_steering_i_rang>0 0</left_steering_i_rang>
-                <right_steering_pid_gain>10000 100 10</right_steering_pid_gain>
-                <right_steering_i_rang>0 0</right_steering_i_rang>
-                <linear_velocity_pid_gain>0.5 10 0.001</linear_velocity_pid_gain>
-                <linear_velocity_i_range>0 0</linear_velocity_i_range>
-                <max_steer>0.523598767</max_steer>
+                <!-- Physical properties -->
                 <wheel_separation>0.172</wheel_separation>
                 <wheel_diameter>0.09</wheel_diameter>
+                <max_steer>0.523598767</max_steer>
                 <max_wheel_torque>20</max_wheel_torque>
                 <max_wheel_acceleration>1.0</max_wheel_acceleration>
-                <command_topic>cmd_vel</command_topic>
-                <publish_odom>true</publish_odom>
-                <publish_odom_tf>true</publish_odom_tf>
-                <publish_wheel_tf>true</publish_wheel_tf>
-                <odometry_topic>odom</odometry_topic>
-                <odometry_frame>odom</odometry_frame>
-                <robot_base_frame>base_footprint</robot_base_frame>
-                <odometry_source>1</odometry_source>
+                <!-- ROS 2 integration -->
+                <ros>
+                    <remapping>~/cmd_vel:=/cmd_vel</remapping>
+                    <remapping>~/odom:=/odom</remapping>
+                </ros>
             </plugin>
         </gazebo>

File: src/limo_ros2/limo_car/gazebo/sensor.xacro (robot description, xacro)
@@ -65,12 +65,12 @@
                     </noise>
                 </ray>
-                <plugin name="gazebo_ros_laser_sensor" filename="libgazebo_ros_ray_sensor.so">
+                <plugin name="gz::sim::systems::RaySensor"
+                            filename="libgz-sim-ray-sensor-system.so">
                     <ros>
-                        <namespace>/</namespace>
-                        <remapping>~/out:=scan</remapping>
+                        <remapping>~/scan:=/scan</remapping>
                     </ros>
-                    <output_type>sensor_msgs/LaserScan</output_type>
+                    <output_type>sensor_msgs/msg/LaserScan</output_type>
                     <min_intensity>150.0</min_intensity>
-                </plugin>
+                    </plugin>
             </sensor>
         </gazebo>
@@ -134,19 +134,19 @@
                     </clip>
                 </camera>
-                <plugin name="gazebo_ros_depth_camera_sensor" filename="libgazebo_ros_camera.so">
+                <plugin name="gz::sim::systems::DepthCamera"
+                            filename="libgz-sim-depth-camera-system.so">
                     <ros>
-<!--                         <namespace>${frame_prefix}</namespace>-->
-                        <remapping>${frame_prefix}/image_raw:=rgb/image_raw</remapping>
-                        <remapping>${frame_prefix}/image_depth:=depth/image_raw</remapping>
-                        <remapping>${frame_prefix}/camera_info:=rgb/camera_info</remapping>
-                        <remapping>${frame_prefix}/camera_info_depth:=depth/camera_info</remapping>
-                        <remapping>${frame_prefix}/points:=depth/points</remapping>
+                        <remapping>~/image:=rgb/image_raw</remapping>
+                        <remapping>~/depth_image:=depth/image_raw</remapping>
+                        <remapping>~/camera_info:=rgb/camera_info</remapping>
+                        <remapping>~/depth_camera_info:=depth/camera_info</remapping>
+                        <remapping>~/points:=depth/points</remapping>
                     </ros>
                     <camera_name>${frame_prefix}</camera_name>
                     <frame_name>${frame_prefix}_frame_optical</frame_name>
-                    <hack_baseline>0.07</hack_baseline>
+                    <baseline>0.07</baseline>
                     <min_depth>0.001</min_depth>
                     <max_depth>300.0</max_depth>
-                </plugin>
+                    </plugin>
             </sensor>
         </gazebo>
@@ -193,12 +193,13 @@
                 <topic>__default_topic__</topic>
                 <pose>0 0 0 0 0 0</pose>
-                <plugin filename="libgazebo_ros_imu_sensor.so" name="imu_plugin">
-                    <topicName>/limo/imu</topicName>
-                    <bodyName>${frame_prefix}_link</bodyName>
-                    <updateRateHZ>100.0</updateRateHZ>
-                    <gaussianNoise>0.001</gaussianNoise>
-                    <xyzOffset>0 0 0</xyzOffset>
-                    <rpyOffset>0 0 0</rpyOffset>
-                    <frameName>${frame_prefix}_link</frameName>
+                <plugin name="gz::sim::systems::Imu"
+                                filename="libgz-sim-imu-system.so">
+                        <ros>
+                            <remapping>~/imu:=/limo/imu</remapping>
+                        </ros>
+                        <topic>/limo/imu</topic>
+                        <update_rate>100.0</update_rate>
+                        <gaussian_noise>0.001</gaussian_noise>
+                        <frame_id>${frame_prefix}_link</frame_id>
                 </plugin>
             </sensor>

File: src/limo_ros2/limo_description/urdf/limo_four_diff.xacro (robot description, xacro)
@@ -2,5 +2,4 @@
 <robot name="limo_four_diff" xmlns:xacro="http://ros.org/wiki/xacro">
     <xacro:include filename="$(find limo_description)/urdf/limo_xacro.xacro" />
-    <!-- <xacro:include filename="$(find limo_description)/urdf/limo_four_diff_2.gazebo" /> -->
     <!-- Variables -->
     <xacro:property name="M_PI" value="3.14159"/>
@@ -15,10 +14,10 @@
     <xacro:property name="wheel_length" value="0.045" />
     <xacro:property name="wheel_radius" value="0.045" />
-  <link name="base_footprint"/>
-  <joint name="base_joint" type="fixed">
-    <parent link="base_footprint"/>
-    <child link="base_link"/>
-    <origin xyz="0.0 0.0 0.15" rpy="0 0 0"/>
-  </joint>
+    <link name="base_footprint"/>
+    <joint name="base_joint" type="fixed">
+        <parent link="base_footprint"/>
+        <child link="base_link"/>
+        <origin xyz="0.0 0.0 0.15" rpy="0 0 0"/>
+    </joint>
     <!-- Base link -->
     <link name="base_link">
@@ -30,9 +29,8 @@
         </visual>
         <collision>
-            <!--origin xyz="0 0 -0.15" rpy="0 0 1.57" /-->
             <origin xyz="0 0 0" rpy="0 0 0" />
-          <geometry>
-              <box size="${base_x_size} ${base_y_size} ${base_z_size}"/>
-          </geometry>
+            <geometry>
+                <box size="${base_x_size} ${base_y_size} ${base_z_size}"/>
+            </geometry>
         </collision>
     </link>
@@ -51,4 +49,5 @@
         <child link="inertial_link" />
     </joint>
+    <!-- Sensors -->
     <xacro:limo_laser parent_prefix="base_link" frame_prefix="laser">
         <origin xyz="0.103 0 -0.034" rpy="0 0 0"/>
@@ -60,6 +59,7 @@
         <origin xyz="0.0 0 -0.1" rpy="0 0 0"/>
     </xacro:limo_imu>
+    <!-- Wheels (links from macro) -->
     <xacro:limo_wheel parent_prefix="base_link" wheel_prefix="front_left" reflect="1">
-        <origin xyz="${wheelbase/2} ${track/2} ${wheel_vertical_offset}" rpy="0 0  0" />
+        <origin xyz="${wheelbase/2} ${track/2} ${wheel_vertical_offset}" rpy="0 0 0" />
     </xacro:limo_wheel>
     <xacro:limo_wheel parent_prefix="base_link" wheel_prefix="front_right" reflect="-1">
@@ -72,207 +72,103 @@
         <origin xyz="${-wheelbase/2} ${-track/2} ${wheel_vertical_offset}" rpy="${M_PI} 0 0" />
     </xacro:limo_wheel>
+    <!-- Gazebo IMU -->
     <gazebo reference="imu_link">
-    <gravity>true</gravity>
-    <sensor name="twr_imu" type="imu">
-      <always_on>true</always_on>
-      <update_rate>100</update_rate>
-      <visualize>true</visualize>
-      <imu>
-        <orientation>
-          <x>
-            <noise type="gaussian">
-              <mean>0.0</mean>
-              <stddev>2e-3</stddev>
-            </noise>
-          </x>
-          <y>
-            <noise type="gaussian">
-              <mean>0.0</mean>
-              <stddev>2e-3</stddev>
-            </noise>
-          </y>
-          <z>
-            <noise type="gaussian">
-              <mean>0.0</mean>
-              <stddev>2e-3</stddev>
-            </noise>
-          </z>
-        </orientation>
-        <angular_velocity>
-          <x>
-            <noise type="gaussian">
-              <mean>0.0</mean>
-              <stddev>2e-4</stddev>
-            </noise>
-          </x>
-          <y>
-            <noise type="gaussian">
-              <mean>0.0</mean>
-              <stddev>2e-4</stddev>
-            </noise>
-          </y>
-          <z>
-            <noise type="gaussian">
-              <mean>0.0</mean>
-              <stddev>2e-4</stddev>
-            </noise>
-          </z>
-        </angular_velocity>
-        <linear_acceleration>
-          <x>
-            <noise type="gaussian">
-              <mean>0.0</mean>
-              <stddev>1.7e-2</stddev>
-            </noise>
-          </x>
-          <y>
-            <noise type="gaussian">
-              <mean>0.0</mean>
-              <stddev>1.7e-2</stddev>
-            </noise>
-          </y>
-          <z>
-            <noise type="gaussian">
-              <mean>0.0</mean>
-              <stddev>1.7e-2</stddev>
-            </noise>
-          </z>
-        </linear_acceleration>
-      </imu>
-      <plugin name="two_wheeled_robot_imu" filename="libgazebo_ros_imu_sensor.so">
-        <initial_orientation_as_reference>false</initial_orientation_as_reference>
-        <frame_name>imu_link</frame_name>
-        <ros>
-          <namespace>/imu</namespace>
-          <remapping>~/out:=data</remapping>
-        </ros>
+      <gravity>true</gravity>
+      <sensor name="twr_imu" type="imu">
+        <always_on>true</always_on>
+        <update_rate>100</update_rate>
+        <visualize>true</visualize>
+        <imu>
+          <orientation>
+            <x><noise type="gaussian"><mean>0.0</mean><stddev>2e-3</stddev></noise></x>
+            <y><noise type="gaussian"><mean>0.0</mean><stddev>2e-3</stddev></noise></y>
+            <z><noise type="gaussian"><mean>0.0</mean><stddev>2e-3</stddev></noise></z>
+          </orientation>
+          <angular_velocity>
+            <x><noise type="gaussian"><mean>0.0</mean><stddev>2e-4</stddev></noise></x>
+            <y><noise type="gaussian"><mean>0.0</mean><stddev>2e-4</stddev></noise></y>
+            <z><noise type="gaussian"><mean>0.0</mean><stddev>2e-4</stddev></noise></z>
+          </angular_velocity>
+          <linear_acceleration>
+            <x><noise type="gaussian"><mean>0.0</mean><stddev>1.7e-2</stddev></noise></x>
+            <y><noise type="gaussian"><mean>0.0</mean><stddev>1.7e-2</stddev></noise></y>
+            <z><noise type="gaussian"><mean>0.0</mean><stddev>1.7e-2</stddev></noise></z>
+          </linear_acceleration>
+        </imu>
+        <plugin name="gz::sim::systems::Imu" filename="libgz-sim8-imu-system.so">
+          <ros>
+            <remapping>~/out:=/imu/data</remapping>
+          </ros>
+        </plugin>
+      </sensor>
+    </gazebo>
+    <!-- Gazebo Laser -->
+    <gazebo reference="laser_link">
+      <sensor name="laser" type="ray">
+        <always_on>true</always_on>
+        <visualize>true</visualize>
+        <update_rate>10</update_rate>
+        <ray>
+          <scan>
+            <horizontal>
+              <samples>120</samples>
+              <resolution>1.0</resolution>
+              <min_angle>-3.14159</min_angle>
+              <max_angle>3.14159</max_angle>
+            </horizontal>
+          </scan>
+          <range>
+            <min>0.3</min>
+            <max>15.0</max>
+            <resolution>0.015</resolution>
+          </range>
+          <noise>
+            <type>gaussian</type>
+            <mean>0.0</mean>
+            <stddev>0.01</stddev>
+          </noise>
+        </ray>
+        <plugin name="scan" filename="libgz-sim8-ros2-ray-sensor-system.so">
+          <ros>
+            <remapping>~/out:=scan</remapping>
+          </ros>
+          <output_type>sensor_msgs/LaserScan</output_type>
+          <frame_name>laser_link</frame_name>
+        </plugin>
+      </sensor>
+    </gazebo>
+    <!-- Wheel contact properties -->
+    <gazebo reference="front_left_wheel_link">
+      <mu1>100</mu1><mu2>100</mu2><kp>10000000.0</kp><kd>1.0</kd><minDepth>0.01</minDepth><fdir1>1 0 0</fdir1>
+    </gazebo>
+    <gazebo reference="front_right_wheel_link">
+      <mu1>100</mu1><mu2>100</mu2><kp>10000000.0</kp><kd>1.0</kd><minDepth>0.01</minDepth><fdir1>1 0 0</fdir1>
+    </gazebo>
+    <gazebo reference="rear_left_wheel_link">
+      <mu1>100</mu1><mu2>100</mu2><kp>10000000.0</kp><kd>1.0</kd><minDepth>0.01</minDepth><fdir1>1 0 0</fdir1>
+    </gazebo>
+    <gazebo reference="rear_right_wheel_link">
+      <mu1>100</mu1><mu2>100</mu2><kp>10000000.0</kp><kd>1.0</kd><minDepth>0.01</minDepth><fdir1>1 0 0</fdir1>
+    </gazebo>
+    <!-- DiffDrive Plugin -->
+    <gazebo>
+      <plugin name="gz::sim::systems::DiffDrive" filename="libgz-sim8-diff-drive-system.so">
+        <update_rate>50</update_rate>
+        <!-- Left wheels -->
+        <left_joint>front_left_wheel</left_joint>
+        <left_joint>rear_left_wheel</left_joint>
+        <!-- Right wheels -->
+        <right_joint>front_right_wheel</right_joint>
+        <right_joint>rear_right_wheel</right_joint>
+        <!-- Wheel geometry -->
+        <wheel_separation>0.172</wheel_separation>
+        <wheel_radius>0.045</wheel_radius>
+        <!-- ROS interface -->
+        <topic>cmd_vel</topic>
+        <odom_topic>odom</odom_topic>
+        <!-- Frames -->
+        <odom_frame>odom</odom_frame>
+        <base_frame>base_footprint</base_frame>
       </plugin>
-    </sensor>
-</gazebo>
-<gazebo reference="laser_link">
-    <sensor name="laser" type="ray">
-      <always_on>true</always_on>
-      <visualize>true</visualize>
-      <update_rate>10</update_rate>
-      <ray>
-        <scan>
-          <horizontal>
-            <samples>120</samples>
-            <resolution>1.000000</resolution>
-            <min_angle>-3.14159</min_angle>
-            <max_angle>3.14159</max_angle>
-          </horizontal>
-        </scan>
-        <range>
-          <min>0.3</min>
-          <max>15.0</max>
-          <resolution>0.015</resolution>
-        </range>
-        <noise>
-          <type>gaussian</type>
-          <mean>0.0</mean>
-          <stddev>0.01</stddev>
-        </noise>
-      </ray>
-      <plugin name="scan" filename="libgazebo_ros_ray_sensor.so">
-        <ros>
-          <remapping>~/out:=scan</remapping>
-        </ros>
-        <output_type>sensor_msgs/LaserScan</output_type>
-        <frame_name>laser_link</frame_name>
-      </plugin>
-    </sensor>
-  </gazebo>
-    <gazebo reference="front_left_wheel">
-        <mu1>100</mu1>
-        <mu2>100</mu2>
-        <kp>10000000.0</kp>
-        <kd>1.0</kd>
-        <minDepth>0.01</minDepth>
-        <fdir1>1 0 0</fdir1>
-        <maxContacts value="64"/>
     </gazebo>
-    <gazebo reference="front_right_wheel">
-        <mu1>100</mu1>
-        <mu2>100</mu2>
-        <kp>10000000.0</kp>
-        <kd>1.0</kd>
-        <minDepth>0.01</minDepth>
-        <fdir1>1 0 0</fdir1>
-        <maxContacts value="64"/>
-    </gazebo>
-    <gazebo reference="rear_left_wheel">
-        <mu1>100</mu1>
-        <mu2>100</mu2>
-        <kp>10000000.0</kp>
-        <kd>1.0</kd>
-        <minDepth>0.01</minDepth>
-        <fdir1>1 0 0</fdir1>
-        <maxContacts value="64"/>
-    </gazebo>
-    <gazebo reference="rear_right_wheel">
-        <mu1>100</mu1>
-        <mu2>100</mu2>
-        <kp>10000000.0</kp>
-        <kd>1.0</kd>
-        <minDepth>0.01</minDepth>
-        <fdir1>1 0 0</fdir1>
-        <maxContacts value="64"/>
-    </gazebo>
-    <gazebo>
-        <plugin name="four_diff_controller" filename="libgazebo_ros_diff_drive.so">
-        <update_rate>50</update_rate>
-        <num_wheel_pairs>2</num_wheel_pairs>
-        <left_joint>front_left_wheel</left_joint>
-        <right_joint>front_right_wheel</right_joint>
-        <left_joint>rear_left_wheel</left_joint>
-        <right_joint>rear_right_wheel</right_joint>
-        <wheel_separation>0.172</wheel_separation>
-        <wheel_diameter>0.09</wheel_diameter>
-        <max_wheel_torque>20</max_wheel_torque>
-        <max_wheel_acceleration>1.0</max_wheel_acceleration>
-        <command_topic>cmd_vel</command_topic>
-        <publish_odom>true</publish_odom>
-        <publish_odom_tf>true</publish_odom_tf>
-        <publish_wheel_tf>true</publish_wheel_tf>
-        <odometry_topic>odom</odometry_topic>
-        <odometry_frame>odom</odometry_frame>
-        <robot_base_frame>base_footprint</robot_base_frame>
-        <odometry_source>1</odometry_source>
-        <ros>
-            <remapping>odom:=/odometry</remapping>
-        </ros>
-        </plugin>
-    </gazebo>
-        <!-- <gazebo reference="depth_camera_link">
-          <sensor name="sensor_camera" type="depth">
-            <pose>0.0 0.0 0.0 0.0 0.0 0.0</pose>
-            <always_on>0</always_on>
-            <update_rate>1</update_rate>
-            <camera name="limo_camera">
-              <distortion>
-                <k1>0.1</k1>
-                <k2>0.2</k2>
-                <k3>0.3</k3>
-                <p1>0.4</p1>
-                <p2>0.5</p2>
-                <center>0.5 0.5</center>
-              </distortion>
-            </camera>
-            <plugin name="gazebo_ros_depth_camera_sensor" filename="libgazebo_ros_camera.so">
-              <ros>
-                <namespace>/limo</namespace>
-                <argument>limo_camera/image_raw:=limo_camera/image</argument>
-                <argument>limo_camera/image_depth:=limo_camera/depth/camera_image_depth</argument>
-                <argument>limo_camera/camera_info:=limo_camera/camera_info_raw</argument>
-                <argument>limo_camera/camera_info_depth:=limo_camera/camera_info_depth</argument>
-                <argument>limo_camera/points:=limo_camera/camera_points</argument>
-              </ros>
-              <camera_name>depth_camera_link</camera_name>
-              <frame_name>depth_camera_link</frame_name>
-              <hack_baseline>0.07</hack_baseline>
-              <min_depth>0.001</min_depth>
-            </plugin>
-        </sensor>
-          </gazebo> -->
 </robot>
